Commit message: scripts and configs

File: system_files/velma_robot - velma_description - robots/50s035x0018z/velma.urdf.xacro (robot description, xacro)
@@ -205,4 +205,7 @@
   </xacro:if>
   <xacro:property name="M_PI" value="3.1415926535897931" />
+  <xacro:property name="RADIANS" value="0.872664626" />
+  <xacro:property name="X_VAL" value="0.07430631098" />
+  <xacro:property name="Z_VAL" value="-0.02593420362" />
   <link name="world" />
   <!-- static connection between the world frame and the map frame -->
@@ -335,5 +338,5 @@
     <child link="right_FtSensorLink"/>
                                   <!-- 39.56 degrees -->
-    <origin xyz="0.08131727983 0.0 -0.00799642866" rpy="0 ${M_PI/4} 0"/>
+    <origin xyz="${X_VAL} 0.0 ${Z_VAL}" rpy="0 ${RADIANS} 0"/>
     <axis xyz="0 0 1"/>
                           <!-- measured max angle is 94.  so upper limit is 94 - start orientation (42 degrees)-->
@@ -362,5 +365,5 @@
     <child link="left_FtSensorLink"/>
                                   <!-- 39.56 degrees -->
-    <origin xyz="0.08131727983 0.0 -0.00799642866" rpy="0 ${M_PI/4} 0"/>
+    <origin xyz="${X_VAL} 0.0 ${Z_VAL}" rpy="0 ${RADIANS} 0"/>
     <axis xyz="0 0 1"/>
                           <!-- measured max angle is 94.  so upper limit is 94 - start orientation (42 degrees)-->
